File: rpi_cm3plus_tablet.sch (EAGLE design)
At the start: 2 parts, among them X1 FH12-15S-0.5SH

Commit message: removed tvdac (should be unused)
Connections:
- net 3.3V: no longer PCB1.166/TVDAC
Changed lines of the file:
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@@
 <layer number="201" name="201bmp" color="2" fill="10" visible="no" active="yes"/>
 </layers>
-<schematic xreflabel="%F%N/%S.%C%R" xrefpart="/%S.%C%R">
+<schematic xreflabel="%F%N/%S" xrefpart="/%S.%C%R">
 <attributes>
 </attributes>
@@
 <net name="3.3V" class="0">
 <segment>
-<pinref part="PCB1" gate="G$1" pin="166/TVDAC"/>
-<wire x1="129.54" y1="-73.66" x2="139.7" y2="-73.66" width="0.1524" layer="91"/>
-<label x="139.7" y="-73.66" size="1.27" layer="95" xref="yes"/>
-</segment>
-<segment>
 <pinref part="PCB1" gate="G$1" pin="194/3V3"/>

Commit message: Modified library to include some custom parts and added a basic usb circuit.
Parts:
- added C1: 0.1uF, resistor:C-USC0603K
- added R1, R2: 47K, resistor:R-US_R0603
- added U$1: FSUSB42MUX, e14_Rpi_Compute_RevC:FSUSB42MUX
- added U$2: BSS138-N, e14_Rpi_Compute_RevC:BSS138-N
Connections:
- removed net VBAT: PCB1.197/VBAT, PCB1.198/VBAT, PCB1.199/VBAT, PCB1.200/VBAT
- new net 5V: PCB1.197/VBAT, PCB1.198/VBAT, PCB1.199/VBAT, PCB1.200/VBAT, R2.1, U$2.G
- new net N$3: C1.2, R1.2, U$1.SEL, U$2.D
- new net N$4: U$1.OUTA_DP
- new net N$5: U$1.OUTA_DM
- new net N$6: U$1.OUTB_DP
- new net N$7: U$1.OUTB_DM
- new net USB_DM: PCB1.167/USB_DM**, U$1.IN_DM
- new net USB_DP: PCB1.165/USB_DP**, U$1.IN_DP
- net 3.3V: now also C1.1, R1.1, U$1.VCC
- net GND: now also R2.2, U$1.GND, U$1.OE, U$2.S
Other:
- moved on the sheet: X1-1, X1-10, X1-11, X1-12, X1-13, X1-14, X1-15, X1-2, X1-3, X1-4, X1-5, X1-6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

Commit message: further updates to schematic regarding custom library
Parts:
- PCB1: device e14_Rpi_Compute_RevC:RPI_COMPUTE -> rpi_cm3plus_tablet:RPI_COMPUTE
- U$1: device e14_Rpi_Compute_RevC:FSUSB42MUX -> rpi_cm3plus_tablet:FSUSB42MUX
- U$2: value BSS138-N -> BSS138N; device e14_Rpi_Compute_RevC:BSS138-N -> rpi_cm3plus_tablet:BSS138N
Changed lines of the file:
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@@
 </classes>
 <parts>
-<part name="PCB1" library="e14_Rpi_Compute_RevC" deviceset="RPI_COMPUTE" device=""/>
+<part name="PCB1" library="rpi_cm3plus_tablet" deviceset="RPI_COMPUTE" device=""/>
 <part name="X1" library="con-hirose" deviceset="FH12-15S-0.5S" device="H"/>
-<part name="U$1" library="e14_Rpi_Compute_RevC" deviceset="FSUSB42MUX" device=""/>
+<part name="U$1" library="rpi_cm3plus_tablet" deviceset="FSUSB42MUX" device=""/>
 <part name="R1" library="resistor" deviceset="R-US_" device="R0603" value="47K"/>
 <part name="R2" library="resistor" deviceset="R-US_" device="R0603" value="47K"/>
 <part name="C1" library="resistor" deviceset="C-US" device="C0603K" value="0.1uF"/>
-<part name="U$2" library="e14_Rpi_Compute_RevC" deviceset="BSS138-N" device=""/>
+<part name="U$2" library="rpi_cm3plus_tablet" deviceset="BSS138N" device=""/>
 </parts>
 <sheets>
